Commit message: WS2: trayectoria del 5 con pose real y punto de dibujo en el eje de las ruedas

File: urdf/Robot-Pogyo_Lorona-WS2.xacro (robot description, xacro)
@@ -20,7 +20,7 @@
   </visual>
   <collision>
-    <origin xyz="0 0 0" rpy="0 0 0"/>
+    <origin xyz="0 0 0.0525" rpy="0 0 0"/>
     <geometry>
-      <mesh filename="file://$(find Robot-Pogyo_Lorona-WS2_description)/meshes/base_link.stl" scale="0.001 0.001 0.001"/>
+      <box size="0.22 0.16 0.07"/>
     </geometry>
   </collision>
@@ -41,10 +41,4 @@
     </material>
   </visual>
-  <collision>
-    <origin xyz="-0.0 -0.0 -0.0875" rpy="0 0 0"/>
-    <geometry>
-      <mesh filename="file://$(find Robot-Pogyo_Lorona-WS2_description)/meshes/lidar_1.stl" scale="0.001 0.001 0.001"/>
-    </geometry>
-  </collision>
 </link>
 <link name="camera_1">
@@ -63,10 +57,4 @@
     </material>
   </visual>
-  <collision>
-    <origin xyz="-0.11 -0.0 -0.0575" rpy="0 0 0"/>
-    <geometry>
-      <mesh filename="file://$(find Robot-Pogyo_Lorona-WS2_description)/meshes/camera_1.stl" scale="0.001 0.001 0.001"/>
-    </geometry>
-  </collision>
 </link>
 <link name="caster_1">
@@ -85,8 +73,22 @@
     </material>
   </visual>
+</link>
+<link name="caster_swivel">
+  <inertial>
+    <origin xyz="0 0 0" rpy="0 0 0"/>
+    <mass value="0.010"/>
+    <inertia ixx="1e-6" iyy="1e-6" izz="1e-6" ixy="0.0" iyz="0.0" ixz="0.0"/>
+  </inertial>
+</link>
+<link name="caster_wheel">
+  <inertial>
+    <origin xyz="0 0 0" rpy="0 0 0"/>
+    <mass value="0.050"/>
+    <inertia ixx="1e-6" iyy="1e-6" izz="1e-6" ixy="0.0" iyz="0.0" ixz="0.0"/>
+  </inertial>
   <collision>
-    <origin xyz="-0.0 -0.0 -0.0175" rpy="0 0 0"/>
+    <origin xyz="0 0 0" rpy="0 0 0"/>
     <geometry>
-      <mesh filename="file://$(find Robot-Pogyo_Lorona-WS2_description)/meshes/caster_1.stl" scale="0.001 0.001 0.001"/>
+      <sphere radius="0.0175"/>
     </geometry>
   </collision>
@@ -108,7 +110,7 @@
   </visual>
   <collision>
-    <origin xyz="0.08 0.08 -0.0375" rpy="0 0 0"/>
+    <origin xyz="0.0 -0.01 -0.001" rpy="1.5707963 0 0"/>
     <geometry>
-      <mesh filename="file://$(find Robot-Pogyo_Lorona-WS2_description)/meshes/right_wheel_1.stl" scale="0.001 0.001 0.001"/>
+      <cylinder radius="0.0375" length="0.02"/>
     </geometry>
   </collision>
@@ -130,7 +132,7 @@
   </visual>
   <collision>
-    <origin xyz="0.08 -0.08 -0.0375" rpy="0 0 0"/>
+    <origin xyz="0.0 0.01 -0.001" rpy="1.5707963 0 0"/>
     <geometry>
-      <mesh filename="file://$(find Robot-Pogyo_Lorona-WS2_description)/meshes/left_wheel_1.stl" scale="0.001 0.001 0.001"/>
+      <cylinder radius="0.0375" length="0.02"/>
     </geometry>
   </collision>
@@ -151,4 +153,16 @@
   <child link="caster_1"/>
 </joint>
+<joint name="Caster_Swivel_Joint" type="continuous">
+  <origin xyz="0.06 0 0" rpy="0 0 0"/>
+  <parent link="caster_1"/>
+  <child link="caster_swivel"/>
+  <axis xyz="0 0 1"/>
+</joint>
+<joint name="Caster_Wheel_Joint" type="continuous">
+  <origin xyz="0 0 0" rpy="0 0 0"/>
+  <parent link="caster_swivel"/>
+  <child link="caster_wheel"/>
+  <axis xyz="0 1 0"/>
+</joint>
 <joint name="Right_Joint" type="continuous">
   <origin xyz="-0.08 -0.08 0.0375" rpy="0 0 0"/>
